File: ATlessX/ATlessX.sch (KiCad schematic (older format))
At the start: 21 parts, among them J1 EXT_PWR_SW, J2 ATX, J3 P8, J4 P9, SW1 Power, U1 74LS74, U2 74LS14, U3 L7905

Commit message: Add some footprints
Parts:
- C1, C2: footprint (none) -> Capacitor_THT:CP_Radial_D6.3mm_P2.50mm
- D1, D2: footprint (none) -> Diode_THT:D_DO-35_SOD27_P7.62mm_Horizontal
- D3, D4, D5, D6, D7: footprint (none) -> LED_THT:LED_D3.0mm
- J2: footprint (none) -> Connector_Molex:Molex_Mini-Fit_Jr_5566-20A_2x10_P4.20mm_Vertical
- R1, R2, R3: footprint (none) -> Resistor_THT:R_Axial_DIN0207_L6.3mm_D2.5mm_P10.16mm_Horizontal
- SW1: footprint (none) -> Button_Switch_THT:SW_PUSH_6mm
- U1, U2: footprint (none) -> Package_DIP:DIP-14_W7.62mm_Socket_LongPads
- U3: footprint (none) -> Package_TO_SOT_THT:TO-220-3_Horizontal_TabDown
Changed lines of the file:
@@
 $EndDescr
 $Comp
-L power:GND #PWR?
+L power:GND #PWR0101
 U 1 1 5DD82289
 P 6600 1600
-F 0 "#PWR?" H 6600 1350 50  0001 C CNN
+F 0 "#PWR0101" H 6600 1350 50  0001 C CNN
 F 1 "GND" V 6605 1472 50  0000 R CNN
 F 2 "" H 6600 1600 50  0001 C CNN
@@
 F 0 "U1" H 5700 3628 50  0000 C CNN
 F 1 "74LS74" H 5700 3537 50  0000 C CNN
-F 2 "" H 5700 3150 50  0001 C CNN
+F 2 "Package_DIP:DIP-14_W7.62mm_Socket_LongPads" H 5700 3150 50  0001 C CNN
 F 3 "74xx/74hc_hct74.pdf" H 5700 3150 50  0001 C CNN
 	1    5700 3150
@@
 F 0 "U1" V 5233 1250 50  0000 C CNN
 F 1 "74LS74" V 5324 1250 50  0000 C CNN
-F 2 "" H 5600 1250 50  0001 C CNN
+F 2 "Package_DIP:DIP-14_W7.62mm_Socket_LongPads" H 5600 1250 50  0001 C CNN
 F 3 "74xx/74hc_hct74.pdf" H 5600 1250 50  0001 C CNN
 	3    5600 1250
@@
 F 0 "U2" V 5233 1900 50  0000 C CNN
 F 1 "74LS14" V 5324 1900 50  0000 C CNN
-F 2 "" H 5600 1900 50  0001 C CNN
+F 2 "Package_DIP:DIP-14_W7.62mm_Socket_LongPads" H 5600 1900 50  0001 C CNN
 F 3 "http://www.ti.com/lit/gpn/sn74LS14" H 5600 1900 50  0001 C CNN
 	7    5600 1900
@@
 F 0 "D1" H 1350 2555 50  0000 C CNN
 F 1 "1N4148" H 1350 2464 50  0000 C CNN
-F 2 "" V 1350 2350 50  0001 C CNN
+F 2 "Diode_THT:D_DO-35_SOD27_P7.62mm_Horizontal" V 1350 2350 50  0001 C CNN
 F 3 "~" V 1350 2350 50  0001 C CNN
 	1    1350 2350
@@
 F 0 "R3" H 1159 2896 50  0000 L CNN
 F 1 "470" H 1159 2805 50  0000 L CNN
-F 2 "" H 1100 2850 50  0001 C CNN
+F 2 "Resistor_THT:R_Axial_DIN0207_L6.3mm_D2.5mm_P10.16mm_Horizontal" H 1100 2850 50  0001 C CNN
 F 3 "~" H 1100 2850 50  0001 C CNN
 	1    1100 2850
@@
 F 0 "SW1" V 896 3902 50  0000 R CNN
 F 1 "Power" V 805 3902 50  0000 R CNN
-F 2 "" H 850 4150 50  0001 C CNN
+F 2 "Button_Switch_THT:SW_PUSH_6mm" H 850 4150 50  0001 C CNN
 F 3 "~" H 850 4150 50  0001 C CNN
 	1    850  3950
@@
 F 0 "C2" H 2041 4096 50  0000 L CNN
 F 1 "10uF" H 2041 4005 50  0000 L CNN
-F 2 "" H 1950 4050 50  0001 C CNN
+F 2 "Capacitor_THT:CP_Radial_D6.3mm_P2.50mm" H 1950 4050 50  0001 C CNN
 F 3 "~" H 1950 4050 50  0001 C CNN
 	1    1950 4050
@@
 F 0 "R1" H 909 2396 50  0000 L CNN
 F 1 "10K" H 909 2305 50  0000 L CNN
-F 2 "" H 850 2350 50  0001 C CNN
+F 2 "Resistor_THT:R_Axial_DIN0207_L6.3mm_D2.5mm_P10.16mm_Horizontal" H 850 2350 50  0001 C CNN
 F 3 "~" H 850 2350 50  0001 C CNN
 	1    850  2350
@@
 F 0 "R2" H 1709 2396 50  0000 L CNN
 F 1 "10K" H 1709 2305 50  0000 L CNN
-F 2 "" H 1650 2350 50  0001 C CNN
+F 2 "Resistor_THT:R_Axial_DIN0207_L6.3mm_D2.5mm_P10.16mm_Horizontal" H 1650 2350 50  0001 C CNN
 F 3 "~" H 1650 2350 50  0001 C CNN
 	1    1650 2350
@@
 F 0 "D2" H 1950 2555 50  0000 C CNN
 F 1 "1N4148" H 1950 2464 50  0000 C CNN
-F 2 "" V 1950 2350 50  0001 C CNN
+F 2 "Diode_THT:D_DO-35_SOD27_P7.62mm_Horizontal" V 1950 2350 50  0001 C CNN
 F 3 "~" V 1950 2350 50  0001 C CNN
 	1    1950 2350
@@
 F 0 "C1" H 1441 4096 50  0000 L CNN
 F 1 "1uF" H 1441 4005 50  0000 L CNN
-F 2 "" H 1350 4050 50  0001 C CNN
+F 2 "Capacitor_THT:CP_Radial_D6.3mm_P2.50mm" H 1350 4050 50  0001 C CNN
 F 3 "~" H 1350 4050 50  0001 C CNN
 	1    1350 4050
@@
 	1350 4450 1950 4450
 $Comp
-L power:GND #PWR?
+L power:GND #PWR0102
 U 1 1 5DD84F2D
 P 1350 4750
-F 0 "#PWR?" H 1350 4500 50  0001 C CNN
+F 0 "#PWR0102" H 1350 4500 50  0001 C CNN
 F 1 "GND" V 1355 4622 50  0000 R CNN
 F 2 "" H 1350 4750 50  0001 C CNN
@@
 F 0 "U3" H 8250 1450 50  0000 C CNN
 F 1 "L7905" H 8250 1359 50  0000 C CNN
-F 2 "" H 8250 1400 50  0001 C CIN
+F 2 "Package_TO_SOT_THT:TO-220-3_Horizontal_TabDown" H 8250 1400 50  0001 C CIN
 F 3 "http://www.st.com/content/ccc/resource/technical/document/datasheet/c9/16/86/41/c7/2b/45/f2/CD00000450.pdf/files/CD00000450.pdf/jcr:content/translations/en.CD00000450.pdf" H 8250 1600 50  0001 C CNN
 	1    8250 1600
@@
 $EndComp
 $Comp
-L power:GND #PWR?
+L power:GND #PWR0103
 U 1 1 5DDA0489
 P 8250 1100
-F 0 "#PWR?" H 8250 850 50  0001 C CNN
+F 0 "#PWR0103" H 8250 850 50  0001 C CNN
 F 1 "GND" V 8255 972 50  0000 R CNN
 F 2 "" H 8250 1100 50  0001 C CNN
@@
 -5V Regulator
 $Comp
-L power:GND #PWR?
+L power:GND #PWR0104
 U 1 1 5DDA6B94
 P 9700 1000
-F 0 "#PWR?" H 9700 750 50  0001 C CNN
+F 0 "#PWR0104" H 9700 750 50  0001 C CNN
 F 1 "GND" V 9705 872 50  0000 R CNN
 F 2 "" H 9700 1000 50  0001 C CNN
@@
 F 0 "D3" V 9200 2550 50  0000 L CNN
 F 1 "5VSB" V 9200 2750 50  0000 L CNN
-F 2 "" V 9700 1750 50  0001 C CNN
+F 2 "LED_THT:LED_D3.0mm" V 9700 1750 50  0001 C CNN
 F 3 "~" V 9700 1750 50  0001 C CNN
 	1    9700 1750
@@
 F 0 "D4" V 9400 2450 50  0000 L CNN
 F 1 "+5V" V 9400 2650 50  0000 L CNN
-F 2 "" V 9800 1750 50  0001 C CNN
+F 2 "LED_THT:LED_D3.0mm" V 9800 1750 50  0001 C CNN
 F 3 "~" V 9800 1750 50  0001 C CNN
 	1    9800 1750
@@
 F 0 "D5" V 9600 2350 50  0000 L CNN
 F 1 "+12V" V 9600 2550 50  0000 L CNN
-F 2 "" V 9900 1750 50  0001 C CNN
+F 2 "LED_THT:LED_D3.0mm" V 9900 1750 50  0001 C CNN
 F 3 "~" V 9900 1750 50  0001 C CNN
 	1    9900 1750
@@
 F 0 "D6" V 10200 2250 50  0000 L CNN
 F 1 "-12V" V 10200 2450 50  0000 L CNN
-F 2 "" V 10000 1750 50  0001 C CNN
+F 2 "LED_THT:LED_D3.0mm" V 10000 1750 50  0001 C CNN
 F 3 "~" V 10000 1750 50  0001 C CNN
 	1    10000 1750
@@
 F 0 "D7" V 10200 2150 50  0000 L CNN
 F 1 "-5V" V 10200 2350 50  0000 L CNN
-F 2 "" V 10100 1750 50  0001 C CNN
+F 2 "LED_THT:LED_D3.0mm" V 10100 1750 50  0001 C CNN
 F 3 "~" V 10100 1750 50  0001 C CNN
 	1    10100 1750
@@
 	9700 1850 9700 2150
 $Comp
-L power:VCC #PWR?
+L power:VCC #PWR0105
 U 1 1 5DDB34E7
 P 9800 1950
-F 0 "#PWR?" H 9800 1800 50  0001 C CNN
+F 0 "#PWR0105" H 9800 1800 50  0001 C CNN
 F 1 "VCC" H 9800 1950 50  0000 C CNN
 F 2 "" H 9800 1950 50  0001 C CNN
@@
 F 0 "J2" H 9050 4267 50  0000 C CNN
 F 1 "ATX" H 9050 4176 50  0000 C CNN
-F 2 "" H 9000 3650 50  0001 C CNN
+F 2 "Connector_Molex:Molex_Mini-Fit_Jr_5566-20A_2x10_P4.20mm_Vertical" H 9000 3650 50  0001 C CNN
 F 3 "~" H 9000 3650 50  0001 C CNN
 	1    9000 3650
@@
 $EndComp
 $Comp
-L power:GND #PWR?
+L power:GND #PWR0106
 U 1 1 5DD98234
 P 1300 1350
-F 0 "#PWR?" H 1300 1100 50  0001 C CNN
+F 0 "#PWR0106" H 1300 1100 50  0001 C CNN
 F 1 "GND" H 1305 1177 50  0000 C CNN
 F 2 "" H 1300 1350 50  0001 C CNN
@@
 ~PS_ON
 $Comp
-L power:VCC #PWR?
+L power:VCC #PWR0107
 U 1 1 5DDB3E20
 P 9500 4100
-F 0 "#PWR?" H 9500 3950 50  0001 C CNN
+F 0 "#PWR0107" H 9500 3950 50  0001 C CNN
 F 1 "VCC" V 9517 4228 50  0000 L CNN
 F 2 "" H 9500 4100 50  0001 C CNN
@@
 	9350 4100 9350 4150
 $Comp
-L power:VCC #PWR?
+L power:VCC #PWR0108
 U 1 1 5DDB8B01
 P 8700 3550
-F 0 "#PWR?" H 8700 3400 50  0001 C CNN
+F 0 "#PWR0108" H 8700 3400 50  0001 C CNN
 F 1 "VCC" V 8717 3677 50  0000 L CNN
 F 2 "" H 8700 3550 50  0001 C CNN
@@
 	8700 3550 8800 3550
 $Comp
-L power:VCC #PWR?
+L power:VCC #PWR0109
 U 1 1 5DDBC074
 P 8700 3750
-F 0 "#PWR?" H 8700 3600 50  0001 C CNN
+F 0 "#PWR0109" H 8700 3600 50  0001 C CNN
 F 1 "VCC" V 8717 3877 50  0000 L CNN
 F 2 "" H 8700 3750 50  0001 C CNN
@@
 +12V
 $Comp
-L power:GND #PWR?
+L power:GND #PWR0110
 U 1 1 5DD98944
 P 8050 3650
-F 0 "#PWR?" H 8050 3400 50  0001 C CNN
+F 0 "#PWR0110" H 8050 3400 50  0001 C CNN
 F 1 "GND" V 8055 3522 50  0000 R CNN
 F 2 "" H 8050 3650 50  0001 C CNN
@@
 	8250 3850 8250 3650
 $Comp
-L power:GND #PWR?
+L power:GND #PWR0111
 U 1 1 5DDA0526
 P 10200 3650
-F 0 "#PWR?" H 10200 3400 50  0001 C CNN
+F 0 "#PWR0111" H 10200 3400 50  0001 C CNN
 F 1 "GND" V 10205 3522 50  0000 R CNN
 F 2 "" H 10200 3650 50  0001 C CNN
@@
 PWR_OK
 $Comp
-L power:VCC #PWR?
+L power:VCC #PWR0112
 U 1 1 5DD99954
 P 1750 5750
-F 0 "#PWR?" H 1750 5600 50  0001 C CNN
+F 0 "#PWR0112" H 1750 5600 50  0001 C CNN
 F 1 "VCC" V 1767 5878 50  0000 L CNN
 F 2 "" H 1750 5750 50  0001 C CNN
@@
 -12V
 $Comp
-L power:GND #PWR?
+L power:GND #PWR0113
 U 1 1 5DDA43EF
 P 1750 6100
-F 0 "#PWR?" H 1750 5850 50  0001 C CNN
+F 0 "#PWR0113" H 1750 5850 50  0001 C CNN
 F 1 "GND" V 1755 5972 50  0000 R CNN
 F 2 "" H 1750 6100 50  0001 C CNN
@@
 	1400 6100 1400 6150
 $Comp
-L power:GND #PWR?
+L power:GND #PWR0114
 U 1 1 5DDACF0F
 P 3500 5700
-F 0 "#PWR?" H 3500 5450 50  0001 C CNN
+F 0 "#PWR0114" H 3500 5450 50  0001 C CNN
 F 1 "GND" V 3505 5572 50  0000 R CNN
 F 2 "" H 3500 5700 50  0001 C CNN
@@
 -5V
 $Comp
-L power:VCC #PWR?
+L power:VCC #PWR0115
 U 1 1 5DDB7431
 P 3500 6050
-F 0 "#PWR?" H 3500 5900 50  0001 C CNN
+F 0 "#PWR0115" H 3500 5900 50  0001 C CNN
 F 1 "VCC" V 3517 6178 50  0000 L CNN
 F 2 "" H 3500 6050 50  0001 C CNN

Commit message: Add footprintd
Parts:
- J1: footprint (none) -> Connector_PinHeader_2.54mm:PinHeader_1x02_P2.54mm_Vertical
- J3, J4: footprint (none) -> Connector_Molex:Molex_Micro-Latch_53253-0670_1x06_P2.00mm_Vertical
Changed lines of the file:
@@
 F 0 "J1" H 1056 1328 50  0000 C CNN
 F 1 "EXT_PWR_SW" H 1056 1237 50  0000 C CNN
-F 2 "" H 950 1150 50  0001 C CNN
+F 2 "Connector_PinHeader_2.54mm:PinHeader_1x02_P2.54mm_Vertical" H 950 1150 50  0001 C CNN
 F 3 "~" H 950 1150 50  0001 C CNN
 	1    950  1150
@@
 F 0 "J3" H 1206 6228 50  0000 C CNN
 F 1 "P8" H 1206 6137 50  0000 C CNN
-F 2 "" H 1100 5850 50  0001 C CNN
+F 2 "Connector_Molex:Molex_Micro-Latch_53253-0670_1x06_P2.00mm_Vertical" H 1100 5850 50  0001 C CNN
 F 3 "~" H 1100 5850 50  0001 C CNN
 	1    1100 5850
@@
 F 0 "J4" H 2956 6228 50  0000 C CNN
 F 1 "P9" H 2956 6137 50  0000 C CNN
-F 2 "" H 2850 5850 50  0001 C CNN
+F 2 "Connector_Molex:Molex_Micro-Latch_53253-0670_1x06_P2.00mm_Vertical" H 2850 5850 50  0001 C CNN
 F 3 "~" H 2850 5850 50  0001 C CNN
 	1    2850 5850

Commit message: Change footprints
Parts:
- J3, J4: footprint Connector_Molex:Molex_Micro-Latch_53253-0670_1x06_P2.00mm_Vertical -> Connector_Molex:Molex_KK-254_AE-6410-06A_1x06_P2.54mm_Vertical
Changed lines of the file:
@@
 F 0 "J3" H 1206 6228 50  0000 C CNN
 F 1 "P8" H 1206 6137 50  0000 C CNN
-F 2 "Connector_Molex:Molex_Micro-Latch_53253-0670_1x06_P2.00mm_Vertical" H 1100 5850 50  0001 C CNN
+F 2 "Connector_Molex:Molex_KK-254_AE-6410-06A_1x06_P2.54mm_Vertical" H 1100 5850 50  0001 C CNN
 F 3 "~" H 1100 5850 50  0001 C CNN
 	1    1100 5850
@@
 F 0 "J4" H 2956 6228 50  0000 C CNN
 F 1 "P9" H 2956 6137 50  0000 C CNN
-F 2 "Connector_Molex:Molex_Micro-Latch_53253-0670_1x06_P2.00mm_Vertical" H 2850 5850 50  0001 C CNN
+F 2 "Connector_Molex:Molex_KK-254_AE-6410-06A_1x06_P2.54mm_Vertical" H 2850 5850 50  0001 C CNN
 F 3 "~" H 2850 5850 50  0001 C CNN
 	1    2850 5850
