File: ATlessX/ATlessX.kicad_pcb (KiCad board)
At the start: 4 copper layers, 90.2 x 73.7 mm, 27 parts, among them J1 EXT_PWR_SW, J2 ATX, J3 P8, J4 P9, SW1 Power, U1 74LS74, U2 74LS14, U3 L7905

Commit message: Update PCB
Other:
- board text added: "+12V"
- board text added: "+5V"
- board text added: "+5VSB"
- board text added: "-12V"
- board text added: "-5V"
- board text added: "ATlessX"
- board text added: "GND"
- board text added: "PWR_OK"
- board text added: "Project & design by tabaglio@posteo.net"
Changed lines of the file:
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@@
-(kicad_pcb (version 20171130) (host pcbnew 5.1.5+dfsg1-2)
+(kicad_pcb (version 20171130) (host pcbnew "(5.1.4-0-10_14)")
   (general
     (thickness 1.6)
-    (drawings 4)
+    (drawings 23)
     (tracks 272)
     (zones 0)
@@
     (1 In1.Cu power hide)
     (2 In2.Cu power hide)
-    (31 B.Cu signal)
+    (31 B.Cu signal hide)
     (32 B.Adhes user)
     (33 F.Adhes user)
@@
     (47 F.CrtYd user)
     (48 B.Fab user)
-    (49 F.Fab user)
+    (49 F.Fab user hide)
   )
   (setup
@@
     (descr "Molex KK-254 Interconnect System, old/engineering part number: AE-6410-06A example for new part number: 22-27-2061, 6 Pins (http://www.molex.com/pdm_docs/sd/022272021_sd.pdf), generated with kicad-footprint-generator")
     (tags "connector Molex KK-254 side entry")
-    (fp_text reference J4 (at 6.35 -4.12) (layer F.SilkS)
+    (fp_text reference J4 (at 6.35 4.064) (layer F.SilkS)
       (effects (font (size 1 1) (thickness 0.15)))
     )
@@
     (descr "Molex KK-254 Interconnect System, old/engineering part number: AE-6410-06A example for new part number: 22-27-2061, 6 Pins (http://www.molex.com/pdm_docs/sd/022272021_sd.pdf), generated with kicad-footprint-generator")
     (tags "connector Molex KK-254 side entry")
-    (fp_text reference J3 (at 6.35 -4.12) (layer F.SilkS)
+    (fp_text reference J3 (at 5.842 4.064) (layer F.SilkS)
       (effects (font (size 1 1) (thickness 0.15)))
     )
@@
     )
   )
+  (gr_text "Project & design by tabaglio@posteo.net" (at 79.502 90.932) (layer F.SilkS)
+    (effects (font (size 1 1) (thickness 0.15) italic))
+  )
+  (gr_text -5V (at 120.65 81.28 90) (layer F.SilkS)
+    (effects (font (size 1 1) (thickness 0.15)))
+  )
+  (gr_text +5V (at 128.27 81.28 90) (layer F.SilkS)
+    (effects (font (size 1 1) (thickness 0.15)))
+  )
+  (gr_text +5V (at 125.73 81.28 90) (layer F.SilkS)
+    (effects (font (size 1 1) (thickness 0.15)))
+  )
+  (gr_text +5V (at 123.19 81.28 90) (layer F.SilkS)
+    (effects (font (size 1 1) (thickness 0.15)))
+  )
+  (gr_text GND (at 118.11 81.28 90) (layer F.SilkS)
+    (effects (font (size 1 1) (thickness 0.15)))
+  )
+  (gr_text GND (at 115.57 81.28 90) (layer F.SilkS)
+    (effects (font (size 1 1) (thickness 0.15)))
+  )
+  (gr_text GND (at 110.49 81.28 90) (layer F.SilkS)
+    (effects (font (size 1 1) (thickness 0.15)))
+  )
+  (gr_text GND (at 107.95 81.28 90) (layer F.SilkS)
+    (effects (font (size 1 1) (thickness 0.15)))
+  )
+  (gr_text -12V (at 105.41 80.772 90) (layer F.SilkS)
+    (effects (font (size 1 1) (thickness 0.15)))
+  )
+  (gr_text +12V (at 102.87 80.772 90) (layer F.SilkS)
+    (effects (font (size 1 1) (thickness 0.15)))
+  )
+  (gr_text +5V (at 100.33 81.28 90) (layer F.SilkS)
+    (effects (font (size 1 1) (thickness 0.15)))
+  )
+  (gr_text PWR_OK (at 97.79 79.756 90) (layer F.SilkS)
+    (effects (font (size 1 1) (thickness 0.15)))
+  )
+  (gr_text -5V (at 130.048 71.374) (layer F.SilkS)
+    (effects (font (size 1 1) (thickness 0.15)))
+  )
+  (gr_text -12V (at 129.54 66.04) (layer F.SilkS)
+    (effects (font (size 1 1) (thickness 0.15)))
+  )
+  (gr_text +12V (at 129.54 60.96) (layer F.SilkS)
+    (effects (font (size 1 1) (thickness 0.15)))
+  )
+  (gr_text +5V (at 130.048 55.88) (layer F.SilkS)
+    (effects (font (size 1 1) (thickness 0.15)))
+  )
+  (gr_text +5VSB (at 129.286 50.8) (layer F.SilkS)
+    (effects (font (size 1 1) (thickness 0.15)))
+  )
+  (gr_text ATlessX (at 109.22 55.88 90) (layer F.SilkS)
+    (effects (font (size 7 7) (thickness 0.45) italic))
+  )
   (gr_line (start 144.78 19.05) (end 144.78 92.71) (layer Edge.Cuts) (width 0.1))

Commit message: Fix design, update gerbers
Connections:
- D5 pad 2: /12V -> /+12V
- J2 pad 1: Net-(J2-Pad1) -> (no net)
- J2 pad 11: Net-(J2-Pad11) -> (no net)
- J2 pad 18: Net-(J2-Pad18) -> (no net)
- J2 pad 2: Net-(J2-Pad2) -> (no net)
- U1 pad 8: Net-(U1-Pad8) -> (no net)
- U1 pad 9: Net-(U1-Pad9) -> (no net)
- U2 pad 10: Net-(U2-Pad10) -> (no net)
- U2 pad 12: Net-(U2-Pad12) -> (no net)
- U2 pad 8: Net-(U2-Pad8) -> (no net)
Routing:
- net /+12V: track 90.8 -> 96.7 mm
