File: ATlessX/ATnoX-smd-2la.kicad_pcb (KiCad board)
At the start: 2 copper layers, 80 x 47 mm, 31 parts, among them J1 EXT_PWR_SW, J2 ATX, P8 P8, P9 P9, SW1 Power, U1 74LS74, U2 74LS14, U3 L7905

Commit message: Added better continuity between 5VSB and GND top/bottom
Routing:
- net /5VSB: track 149.0 -> 152.0 mm, vias 1 -> 2
- net GND: track 269.6 -> 272.3 mm, vias 0 -> 2
Changed lines of the file:
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@@
     (thickness 1.6)
     (drawings 26)
-    (tracks 322)
+    (tracks 333)
     (zones 0)
     (modules 31)
@@
   (segment (start 152.2 71.12) (end 152.2 76.62) (width 0.5) (layer F.Cu) (net 1))
   (segment (start 113.03 69.76) (end 114.4303 69.76) (width 0.5) (layer F.Cu) (net 1))
+  (segment (start 109.155 85.09) (end 110.49 85.09) (width 0.5) (layer F.Cu) (net 1))
+  (via (at 110.49 85.09) (size 1.2) (drill 0.4) (layers F.Cu B.Cu) (net 1))
+  (via (at 111.76 97.79) (size 1.2) (drill 0.4) (layers F.Cu B.Cu) (net 1))
+  (segment (start 110.7827 98.5716) (end 110.9784 98.5716) (width 0.5) (layer F.Cu) (net 1))
+  (segment (start 110.9784 98.5716) (end 111.76 97.79) (width 0.5) (layer F.Cu) (net 1))
   (segment (start 121.7796 86.3737) (end 121.7162 86.3737) (width 0.25) (layer F.Cu) (net 2))
   (segment (start 121.7162 86.3737) (end 118.745 83.4025) (width 0.25) (layer F.Cu) (net 2))
@@
   (segment (start 172.8426 87.63) (end 173.86 87.63) (width 0.25) (layer F.Cu) (net 4))
   (via (at 107.2649 94.9441) (size 0.8) (layers F.Cu B.Cu) (net 4))
+  (segment (start 105.759 84.741) (end 106.68 85.662) (width 0.25) (layer F.Cu) (net 4))
+  (segment (start 105.759 83.9505) (end 105.759 84.741) (width 0.25) (layer F.Cu) (net 4))
+  (segment (start 106.68 85.662) (end 106.68 86.36) (width 0.25) (layer F.Cu) (net 4))
+  (via (at 106.479 86.378531) (size 0.8) (drill 0.4) (layers F.Cu B.Cu) (net 4))
+  (segment (start 106.68 86.36) (end 106.497531 86.36) (width 0.25) (layer F.Cu) (net 4))
+  (segment (start 106.497531 86.36) (end 106.479 86.378531) (width 0.25) (layer F.Cu) (net 4))
   (segment (start 176.66 87.63) (end 178.0677 87.63) (width 0.25) (layer F.Cu) (net 5))
   (segment (start 176.7475 87.63) (end 178.0677 87.63) (width 0.25) (layer B.Cu) (net 5))

Commit message: Add new revision of board
Other:
- board text added: "rev.1"
Changed lines of the file:
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@@
   (general
     (thickness 1.6)
-    (drawings 26)
+    (drawings 27)
     (tracks 333)
     (zones 0)
@@
     )
   )
+  (gr_text rev.1 (at 167.64 111.76) (layer F.SilkS)
+    (effects (font (size 1 1) (thickness 0.15)))
+  )
   (gr_text tabaglio@posteo.net (at 102.87 86.36 270) (layer B.SilkS)

Commit message: Add rev2 board
Routing:
- net VCC: track 236.3 -> 238.9 mm
Other:
- board text added: "rev.2"
- board text removed: "rev.1"
Changed lines of the file:
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@@
     (thickness 1.6)
     (drawings 27)
-    (tracks 333)
+    (tracks 335)
     (zones 0)
     (modules 31)
@@
     )
   )
-  (gr_text rev.1 (at 167.64 111.76) (layer F.SilkS)
-    (effects (font (size 1 1) (thickness 0.15)))
+  (gr_text rev.2 (at 167.64 111.76) (layer F.SilkS)
+    (effects (font (size 1.5 1.5) (thickness 0.3)))
   )
   (gr_text tabaglio@posteo.net (at 102.87 86.36 270) (layer B.SilkS)
@@
   (segment (start 139.7 85.09) (end 151.13 85.09) (width 0.5) (layer F.Cu) (net 6))
   (segment (start 134.62 90.17) (end 139.7 85.09) (width 0.5) (layer F.Cu) (net 6))
-  (segment (start 176.66 90.17) (end 175.4066 90.17) (width 0.25) (layer F.Cu) (net 7))
-  (segment (start 176.7475 90.17) (end 175.4066 90.17) (width 0.25) (layer B.Cu) (net 7))
-  (via (at 175.4066 90.17) (size 0.8) (layers F.Cu B.Cu) (net 7))
+  (segment (start 175.1929 91.4787) (end 175.1808 91.4908) (width 0.5) (layer F.Cu) (net 6))
+  (segment (start 175.1929 88.8371) (end 175.1929 91.4787) (width 0.5) (layer F.Cu) (net 6))
+  (segment (start 176.66 90.17) (end 177.8 90.17) (width 0.25) (layer F.Cu) (net 7))
+  (via (at 177.8 90.17) (size 0.8) (drill 0.4) (layers F.Cu B.Cu) (net 7))
+  (segment (start 177.8 90.17) (end 176.7475 90.17) (width 0.25) (layer B.Cu) (net 7))
   (segment (start 176.66 92.71) (end 178.0922 92.71) (width 0.25) (layer F.Cu) (net 8))
   (segment (start 176.7475 92.71) (end 178.0922 92.71) (width 0.25) (layer B.Cu) (net 8))
