File: ATnoX/ATnoX-smd.kicad_pcb (KiCad board)
At the start: 4 copper layers, 80 x 47 mm, 41 parts, among them J1 EXT_PWR_SW, J2 ATX, J3 AT, J4 PWR_LED, SW1 Power, U1 74LS74, U2 74LS14, U3 L7905, U4 74HCT4060, U5 74HCT73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

Commit message: Add r3.2 gerbers
Parts:
- D1, D2: value 1N4148 -> LL4148; footprint Diode_SMD:D_SOD-123 -> Diode_SMD:D_MiniMELF
- J1: value EXT_PWR_SW -> Power Switch
- J4: value PWR_LED -> Power LED
- U1: value 74LS74 -> 74HC74
- U2: value 74LS14 -> 74HC14
- U4: value 74HCT4060 -> 74HC4060
- U5: value 74HCT73 -> 74HC73
Routing:
- net Net-(C8-Pad1): track 62.5 -> 41.2 mm
- net /-5V: track 65.7 -> 71.0 mm
- net /-12V: track 85.3 -> 89.8 mm
- net GND: track 418.7 -> 415.8 mm, vias 4 -> 5
Other:
- outline, holes or cut-outs redrawn
- board text added: "rev. 3.2"
- board text removed: "74HC14"
- board text removed: "74HC4060"
- board text removed: "74HC73"
- board text removed: "74HC74"
- board text removed: "7905"
- board text removed: "PWR Led"
- board text removed: "Power Button"
- board text removed: "rev. 3.1"
